File: pcb/XNL.kicad_pcb (KiCad board)
At the start: 2 copper layers, 77.5 x 50.8 mm, 70 parts, among them J1 Conn_01x10_Socket, J10 Conn_01x02_Socket, J11 Conn_01x02_Socket, J12 Conn_01x02_Socket, J13 Conn_01x02_Socket, J14 Conn_01x02_Socket, J15 Conn_01x02_Socket, J16 Conn_01x02_Socket, J17 Conn_01x02_Socket, J18 Conn_01x02_Socket, J19 Conn_01x02_Socket, J2 Conn_01x02_Pin, J20 Conn_01x02_Socket, J21 Conn_01x02_Socket, J22 Conn_01x02_Socket, J23 Conn_01x02_Socket, J24 Conn_01x02_Socket, J25 Conn_01x02_Socket, J26 Conn_01x02_Socket, J27 Conn_01x02_Socket, J28 Conn_01x02_Socket, J29 Conn_01x02_Socket, J3 Conn_01x10_Socket, J30 Conn_01x02_Socket, J31 Conn_01x02_Socket, J32 Conn_01x02_Socket, J33 Conn_01x02_Socket, J4 Conn_02x02_Counter_Clockwise, J5 Conn_02x02_Counter_Clockwise, J6 Conn_02x02_Counter_Clockwise, J7 Conn_02x02_Counter_Clockwise, J8 Conn_02x02_Counter_Clockwise, J9 Conn_02x02_Counter_Clockwise, U1 4077, U2 4077

Commit message: Add reverse polarity protection
Parts:
- added D1: BAT43, Diode_SMD:D_MiniMELF, B.Cu at (157.9, 114.3)
- added D2: BZ5V1, Diode_SMD:D_MiniMELF, B.Cu at (156.2, 118.8)
- added Q1: BUK7880-55A, Package_TO_SOT_SMD:SOT-223-3_TabPin2, B.Cu at (150.5, 119.4)
- added R25: 1k, Resistor_SMD:R_1206_3216Metric, B.Cu at (152.8, 114.3)
- moved FID1 37.8 mm to (149.9, 84.5)
- moved FID3 36.9 mm to (168.3, 84.5)
- moved FID2 35.5 mm to (156.2, 84.5)
Connections:
- J2 pad 2: GND -> Net-(J2-Pin_2)
- J3 pad 1: GND -> Net-(J2-Pin_2)
- J3 pad 10: GND -> Net-(J2-Pin_2)
- J3 pad 2: GND -> Net-(J2-Pin_2)
- J3 pad 3: GND -> Net-(J2-Pin_2)
- J3 pad 4: GND -> Net-(J2-Pin_2)
- J3 pad 5: GND -> Net-(J2-Pin_2)
- J3 pad 6: GND -> Net-(J2-Pin_2)
- J3 pad 7: GND -> Net-(J2-Pin_2)
- J3 pad 8: GND -> Net-(J2-Pin_2)
- J3 pad 9: GND -> Net-(J2-Pin_2)
Routing:
- net Net-(J2-Pin_2): track 0.00 -> 38.9 mm
- net VCC: track 222.6 -> 225.1 mm
- net GND: vias 43 -> 48
- added copper zone on B.Cu, net Net-(D1-A)
- added copper zone on B.Cu, net Net-(J2-Pin_2)
